File: KeyboardMatrix.sch (KiCad schematic (older format))
At the start: 134 parts

Commit message: TypeC
Parts:
- 0,13: footprint MX_Only:MXOnly-1U-Hotswap -> MX_Only:MXOnly-2U-Hotswap
- 1,0, 1,13: footprint MX_Only:MXOnly-1U-Hotswap -> MX_Only:MXOnly-1.5U-Hotswap
- 2,0, 3,11: footprint MX_Only:MXOnly-1U-Hotswap -> MX_Only:MXOnly-1.75U-Hotswap
- 2,12, 3,0: footprint MX_Only:MXOnly-1U-Hotswap -> MX_Only:MXOnly-2.25U-Hotswap
- 4,0, 4,1, 4,2, 4,4, 4,5: footprint MX_Only:MXOnly-1U-Hotswap -> MX_Only:MXOnly-1.25U-Hotswap
- 4,3: footprint MX_Only:MXOnly-1U-Hotswap -> MX_Only:MXOnly-6.25U-Hotswap
- renumbered D1 to D0,0, D6 to D0,1, D46 to D0,10, D51 to D0,11, D56 to D0,12, D61 to D0,13, D66 to D0,14, D11 to D0,2, D16 to D0,3, D20 to D0,4, D24 to D0,5, D29 to D0,6, D33 to D0,7, D37 to D0,8, D41 to D0,9, D2 to D1,0, D7 to D1,1, D47 to D1,10, D52 to D1,11, D57 to D1,12, D62 to D1,13, D67 to D1,14, D12 to D1,2, D17 to D1,3, D21 to D1,4, D25 to D1,5, D30 to D1,6, D34 to D1,7, D38 to D1,8, D42 to D1,9, D3 to D2,0, D8 to D2,1, D48 to D2,10, D53 to D2,11, D58 to D2,12, D63 to D2,13, D13 to D2,2, D18 to D2,3, D22 to D2,4, D26 to D2,5, D31 to D2,6, D35 to D2,7, D39 to D2,8, D43 to D2,9, D4 to D3,0, D9 to D3,1, D49 to D3,10, D54 to D3,11, D59 to D3,12, D64 to D3,13, D14 to D3,2, D19 to D3,3, D23 to D3,4, D27 to D3,5, D32 to D3,6, D36 to D3,7, D40 to D3,8, D44 to D3,9, D5 to D4,0, D10 to D4,1, D15 to D4,2, D28 to D4,3, D45 to D4,4, D50 to D4,5, D55 to D4,6, D60 to D4,7, D65 to D4,8
