File: pardus75.kicad_pcb (KiCad board)
At the start: 2 copper layers, 151 parts, among them J1 USB_C_Receptacle, SW1 SW_Push, U1 AT90USB1286-AU, Y1 16MHz

Commit message: TypeC
Parts:
- removed the J1 at (52.5, 172.2)
- added J1: USB4085-GF-A_REVA, Connector_USB:USB_C_Receptacle_GCT_USB4085, F.Cu at (37.2, -81.7)
- added J1: USB_C_Receptacle, Connector_USB:USB_C_Receptacle_Amphenol_12401548E4-2A, B.Cu at (40.4, -64.8)
- 0,13: footprint MX_Only:MXOnly-1U-Hotswap -> MX_Only:MXOnly-2U-Hotswap; moved to B.Cu
- 1,0, 1,13: footprint MX_Only:MXOnly-1U-Hotswap -> MX_Only:MXOnly-1.5U-Hotswap
- 2,0, 3,11: footprint MX_Only:MXOnly-1U-Hotswap -> MX_Only:MXOnly-1.75U-Hotswap
- 2,12, 3,0: footprint MX_Only:MXOnly-1U-Hotswap -> MX_Only:MXOnly-2.25U-Hotswap
- 4,0, 4,1, 4,2, 4,4, 4,5: footprint MX_Only:MXOnly-1U-Hotswap -> MX_Only:MXOnly-1.25U-Hotswap
- 4,3: footprint MX_Only:MXOnly-1U-Hotswap -> MX_Only:MXOnly-6.25U-Hotswap
- C1, C2, C3, C4, C5, C6, C7, R1, R2, R3, R4, R5, R6, SW1, U1, Y1: moved to B.Cu
- D0,0: renamed from D1; moved to B.Cu
- D0,1: renamed from D6; moved to B.Cu
- D0,10: renamed from D46; moved to B.Cu
- D0,11: renamed from D51; moved to B.Cu
- D0,12: renamed from D56; moved to B.Cu
- D0,13: renamed from D61; moved to B.Cu
- D0,14: renamed from D66; moved to B.Cu
- D0,2: renamed from D11; moved to B.Cu
- D0,3: renamed from D16; moved to B.Cu
- D0,4: renamed from D20; moved to B.Cu
- D0,5: renamed from D24; moved to B.Cu
- D0,6: renamed from D29; moved to B.Cu
- D0,7: renamed from D33; moved to B.Cu
- D0,8: renamed from D37; moved to B.Cu
- D0,9: renamed from D41; moved to B.Cu
- D1,0: renamed from D2; moved to B.Cu
- D1,1: renamed from D7; moved to B.Cu
- D1,10: renamed from D47; moved to B.Cu
- D1,11: renamed from D52; moved to B.Cu
- D1,12: renamed from D57; moved to B.Cu
- D1,13: renamed from D62; moved to B.Cu
- D1,14: renamed from D67; moved to B.Cu
- D1,2: renamed from D12; moved to B.Cu
- D1,3: renamed from D17; moved to B.Cu
- D1,4: renamed from D21; moved to B.Cu
- D1,5: renamed from D25; moved to B.Cu
- D1,6: renamed from D30; moved to B.Cu
- D1,7: renamed from D34; moved to B.Cu
- D1,8: renamed from D38; moved to B.Cu
- D1,9: renamed from D42; moved to B.Cu
- D2,0: renamed from D3; moved to B.Cu
- D2,1: renamed from D8; moved to B.Cu
- D2,10: renamed from D48; moved to B.Cu
- D2,11: renamed from D53; moved to B.Cu
- D2,12: renamed from D58; moved to B.Cu
- D2,13: renamed from D63; moved to B.Cu
- D2,2: renamed from D13; moved to B.Cu
- D2,3: renamed from D18; moved to B.Cu
- D2,4: renamed from D22; moved to B.Cu
- D2,5: renamed from D26; moved to B.Cu
- D2,6: renamed from D31; moved to B.Cu
- D2,7: renamed from D35; moved to B.Cu
- D2,8: renamed from D39; moved to B.Cu
- D2,9: renamed from D43; moved to B.Cu
- D3,0: renamed from D4; moved to B.Cu
- D3,1: renamed from D9; moved to B.Cu
- D3,10: renamed from D49; moved to B.Cu
- D3,11: renamed from D54; moved to B.Cu
- D3,12: renamed from D59; moved to B.Cu
- D3,13: renamed from D64; moved to B.Cu
- D3,2: renamed from D14; moved to B.Cu
- D3,3: renamed from D19; moved to B.Cu
- D3,4: renamed from D23; moved to B.Cu
- D3,5: renamed from D27; moved to B.Cu
- D3,6: renamed from D32; moved to B.Cu
- D3,7: renamed from D36; moved to B.Cu
- D3,8: renamed from D40; moved to B.Cu
- D3,9: renamed from D44; moved to B.Cu
- D4,0: renamed from D5; moved to B.Cu
- D4,1: renamed from D10; moved to B.Cu
- D4,2: renamed from D15; moved to B.Cu
- D4,3: renamed from D28; moved to B.Cu
- D4,4: renamed from D45; moved to B.Cu
- D4,5: renamed from D50; moved to B.Cu
- D4,6: renamed from D55; moved to B.Cu
- D4,7: renamed from D60; moved to B.Cu
- D4,8: renamed from D65; moved to B.Cu
- moved D0,14 322.8 mm to (316.2, -63.5), turned to 180 degrees
- moved 0,14 307.9 mm to (316.5, -58.2), turned to 180 degrees
- moved D1,14 305.8 mm to (316.5, -44.5), turned to 180 degrees
- moved D0,13 300.4 mm to (287.8, -63.5), turned to 180 degrees
- moved D4,7 292.5 mm to (297.2, 12.7), turned to 180 degrees
- moved D2,13 291.4 mm to (316.5, -25.4), turned to 180 degrees
- moved D1,13 275.6 mm to (292.6, -44.5), turned to 180 degrees
- moved D3,13 275.2 mm to (316.5, -6.35), turned to 180 degrees
- moved D0,10 265.9 mm to (221.2, -63.5), turned to 180 degrees
- moved D0,11 264.2 mm to (240.3, -63.5), turned to 180 degrees
- moved D0,12 259.6 mm to (259.1, -63.5), turned to 180 degrees
- moved D4,8 259.4 mm to (316.2, 12.7), turned to 180 degrees
- moved 1,12 257.4 mm to (268.9, -39.1), turned to 180 degrees
- moved 0,13 255.1 mm to (287.9, -58.2), turned to 180 degrees
- moved D2,12 254.8 mm to (285.5, -25.4), turned to 180 degrees
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Connections:
- R1 pad 1: GND -> Net-(J1-PadA5)
- R1 pad 2: Net-(J1-PadA5) -> GND
- R2 pad 1: GND -> Net-(J1-PadB5)
- R2 pad 2: Net-(J1-PadB5) -> GND
Other:
- board outline added: 304.8 x 96.1 mm
