File: pardus75.sch (KiCad schematic (older format))
At the start: 17 parts

Commit message: PCB added
Parts:
- C1, C2, C3, C4, C5, C6, C7: renamed from C?; footprint (none) -> Capacitor_SMD:C_0805_2012Metric_Pad1.15x1.40mm_HandSolder
- J1: renamed from J?; footprint (none) -> Connector_USB:USB_C_Receptacle_Amphenol_12401548E4-2A
- R1, R2, R3, R4, R5, R6: renamed from R?; footprint (none) -> Resistor_SMD:R_0805_2012Metric
- SW1: renamed from SW?; footprint (none) -> Button_Switch_SMD:SW_SPST_SKQG_WithStem
- Y1: renamed from Y?; footprint (none) -> Crystal:Crystal_SMD_3225-4Pin_3.2x2.5mm
- gave numbers to parts that had none: 1

Commit message: TypeC
Parts:
- removed J1: USB_C_Receptacle, Connector_USB:USB_C_Receptacle_Amphenol_12401548E4-2A, symbol Connector:USB_C_Receptacle
- added J1: USB4085-GF-A_REVA, Connector_USB:USB_C_Receptacle_GCT_USB4085, symbol USB4085-GF-A_REVA:USB4085-GF-A_REVA
Connections:
- net +5V: now also J1.A4 (VBUS), J1.A9 (VBUS), J1.B4 (VBUS), J1.B9 (VBUS)
- net D+: now also J1.A6 (DP1), J1.B6 (DP2)
- net D-: now also J1.A7 (DN1), J1.B7 (DN2)
- net GND: now also R1.2, R2.2, J1.A1 (GND), J1.A12 (GND), J1.B1 (GND), J1.B12 (GND), J1.P1 (SHELL), J1.P2 (SHELL), J1.P3 (SHELL), J1.P4 (SHELL); no longer R1.1, R2.1
- new net: J1.A5 (CC1), R1.1
- new net: J1.B5 (CC2), R2.1
Other:
- moved on the sheet: C1, R1, R2
Changed lines of the file:
@@
 D-
-$Comp
-L Device:R_Small R1
-U 1 1 5F469DAA
-P 3950 2700
-F 0 "R1" V 3754 2700 50  0000 C CNN
-F 1 "5K1" V 3845 2700 50  0000 C CNN
-F 2 "Resistor_SMD:R_0805_2012Metric" H 3950 2700 50  0001 C CNN
-F 3 "~" H 3950 2700 50  0001 C CNN
-	1    3950 2700
-	0    1    1    0
-$EndComp
-$Comp
-L Device:R_Small R2
-U 1 1 5F46AD36
-P 3950 3000
-F 0 "R2" V 3754 3000 50  0000 C CNN
-F 1 "5K1" V 3845 3000 50  0000 C CNN
-F 2 "Resistor_SMD:R_0805_2012Metric" H 3950 3000 50  0001 C CNN
-F 3 "~" H 3950 3000 50  0001 C CNN
-	1    3950 3000
-	0    1    1    0
-$EndComp
-$Comp
-L power:GND #PWR0114
-U 1 1 5F46BE27
-P 4250 3000
-F 0 "#PWR0114" H 4250 2750 50  0001 C CNN
-F 1 "GND" H 4255 2827 50  0000 C CNN
-F 2 "" H 4250 3000 50  0001 C CNN
-F 3 "" H 4250 3000 50  0001 C CNN
-	1    4250 3000
-	1    0    0    -1
-$EndComp
-Wire Wire Line
-	4250 3000 4050 3000
-Wire Wire Line
-	4050 2700 4250 2700
-Wire Wire Line
-	4250 2700 4250 3000
-Connection ~ 4250 3000
-Wire Wire Line
-	3850 3000 3650 3000
-Wire Wire Line
-	3650 3000 3650 2800
-Wire Wire Line
-	3650 2800 3150 2800
-Wire Wire Line
-	3850 2700 3150 2700
-$Comp
-L Connector:USB_C_Receptacle J1
-U 1 1 5F4676D7
-P 2550 3500
-F 0 "J1" H 2657 4767 50  0000 C CNN
-F 1 "USB_C_Receptacle" H 2657 4676 50  0000 C CNN
-F 2 "Connector_USB:USB_C_Receptacle_Amphenol_12401548E4-2A" H 2700 3500 50  0001 C CNN
-F 3 "https://www.usb.org/sites/default/files/documents/usb_type-c.zip" H 2700 3500 50  0001 C CNN
-	1    2550 3500
-	1    0    0    -1
-$EndComp
-Text GLabel 3450 3000 2    50   Input ~ 0
-D-
-Wire Wire Line
-	3450 3000 3400 3000
-Wire Wire Line
-	3150 3100 3400 3100
-Wire Wire Line
-	3400 3100 3400 3000
-Connection ~ 3400 3000
-Wire Wire Line
-	3400 3000 3150 3000
-Text GLabel 3450 3300 2    50   Input ~ 0
-D+
-Wire Wire Line
-	3150 3300 3400 3300
-Wire Wire Line
-	3150 3200 3400 3200
-Wire Wire Line
-	3400 3200 3400 3300
-Connection ~ 3400 3300
-Wire Wire Line
-	3400 3300 3450 3300
 $Comp
 L power:+5V #PWR0115
 U 1 1 5F47DE63
-P 4850 2500
-F 0 "#PWR0115" H 4850 2350 50  0001 C CNN
-F 1 "+5V" H 4865 2673 50  0000 C CNN
-F 2 "" H 4850 2500 50  0001 C CNN
-F 3 "" H 4850 2500 50  0001 C CNN
-	1    4850 2500
+P 2050 2050
+F 0 "#PWR0115" H 2050 1900 50  0001 C CNN
+F 1 "+5V" H 2000 2200 50  0000 C CNN
+F 2 "" H 2050 2050 50  0001 C CNN
+F 3 "" H 2050 2050 50  0001 C CNN
+	1    2050 2050
 	1    0    0    -1
 $EndComp
-Wire Wire Line
-	3150 2500 4450 2500
 $Comp
 L power:PWR_FLAG #FLG0101
 U 1 1 5F480213
-P 4600 2500
-F 0 "#FLG0101" H 4600 2575 50  0001 C CNN
-F 1 "PWR_FLAG" H 4600 2673 50  0000 C CNN
-F 2 "" H 4600 2500 50  0001 C CNN
-F 3 "~" H 4600 2500 50  0001 C CNN
-	1    4600 2500
+P 2250 2050
+F 0 "#FLG0101" H 2250 2125 50  0001 C CNN
+F 1 "PWR_FLAG" H 2350 2200 50  0000 C CNN
+F 2 "" H 2250 2050 50  0001 C CNN
+F 3 "~" H 2250 2050 50  0001 C CNN
+	1    2250 2050
 	1    0    0    -1
 $EndComp
-Connection ~ 4600 2500
-Wire Wire Line
-	4600 2500 4850 2500
-$Comp
-L Device:C_Small C1
-U 1 1 5F4810C0
-P 4450 2600
-F 0 "C1" H 4542 2646 50  0000 L CNN
-F 1 "1uF" H 4542 2555 50  0000 L CNN
-F 2 "Capacitor_SMD:C_0805_2012Metric_Pad1.15x1.40mm_HandSolder" H 4450 2600 50  0001 C CNN
-F 3 "~" H 4450 2600 50  0001 C CNN
-	1    4450 2600
-	1    0    0    -1
-$EndComp
-Connection ~ 4450 2500
-Wire Wire Line
-	4450 2500 4600 2500
-$Comp
-L power:GND #PWR0116
-U 1 1 5F48215E
-P 4450 2700
-F 0 "#PWR0116" H 4450 2450 50  0001 C CNN
-F 1 "GND" H 4455 2527 50  0000 C CNN
-F 2 "" H 4450 2700 50  0001 C CNN
-F 3 "" H 4450 2700 50  0001 C CNN
-	1    4450 2700
-	1    0    0    -1
-$EndComp
-$Comp
-L power:PWR_FLAG #FLG0102
-U 1 1 5F482E55
-P 2750 5100
-F 0 "#FLG0102" H 2750 5175 50  0001 C CNN
-F 1 "PWR_FLAG" H 2750 5273 50  0000 C CNN
-F 2 "" H 2750 5100 50  0001 C CNN
-F 3 "~" H 2750 5100 50  0001 C CNN
-	1    2750 5100
-	-1   0    0    1
-$EndComp
-$Comp
-L power:GND #PWR0117
-U 1 1 5F486E4E
-P 3050 5100
-F 0 "#PWR0117" H 3050 4850 50  0001 C CNN
-F 1 "GND" H 3055 4927 50  0000 C CNN
-F 2 "" H 3050 5100 50  0001 C CNN
-F 3 "" H 3050 5100 50  0001 C CNN
-	1    3050 5100
-	1    0    0    -1
-$EndComp
-Wire Wire Line
-	2250 5100 2550 5100
-Wire Wire Line
-	2550 5100 2750 5100
-Connection ~ 2550 5100
-Wire Wire Line
-	2750 5100 3050 5100
-Connection ~ 2750 5100
 $Sheet
 S 3550 5850 2300 1250
@@
 F1 "KeyboardMatrix.sch" 50
 $EndSheet
+Wire Wire Line
+	2050 2050 2250 2050
+Connection ~ 2250 2050
+Wire Wire Line
+	2900 3600 2600 3600
+Connection ~ 2900 3600
+Wire Wire Line
+	3150 3600 3150 3550
+Connection ~ 3150 3600
+Wire Wire Line
+	3150 3600 2900 3600
+Wire Wire Line
+	3150 3650 3150 3600
+Connection ~ 3050 3150
+Wire Wire Line
+	3050 3300 2800 3300
+Wire Wire Line
+	3050 3150 3050 3300
+Wire Wire Line
+	3150 3150 3050 3150
+Wire Wire Line
+	3050 3050 3050 3150
+Wire Wire Line
+	3150 3050 3050 3050
+Wire Wire Line
+	3000 2950 3000 3100
+Connection ~ 3000 2950
+Wire Wire Line
+	3000 2850 3000 2950
+Wire Wire Line
+	3150 2950 3000 2950
+Wire Wire Line
+	3000 3100 2800 3100
+Wire Wire Line
+	3150 2850 3000 2850
+Connection ~ 2500 2750
+Wire Wire Line
+	2500 2650 2500 2750
+Wire Wire Line
+	2800 2650 2500 2650
+Wire Wire Line
+	2800 2750 2500 2750
+Wire Wire Line
+	3150 2650 3000 2650
+Wire Wire Line
+	3150 2750 3000 2750
+Wire Wire Line
+	3150 2450 3150 2050
+Connection ~ 2450 2050
+Wire Wire Line
+	2450 2050 3150 2050
+Wire Wire Line
+	2250 2050 2450 2050
+$Comp
+L USB4085-GF-A_REVA:USB4085-GF-A_REVA J1
+U 1 1 5F52FA63
+P 3450 3050
+F 0 "J1" H 3680 3096 50  0000 L CNN
+F 1 "USB4085-GF-A_REVA" H 3680 3005 50  0000 L CNN
+F 2 "Connector_USB:USB_C_Receptacle_GCT_USB4085" H 3450 3050 50  0001 L BNN
+F 3 "Manufacturer Recommendations" H 3450 3050 50  0001 L BNN
+F 4 "Global Connector Technology" H 3450 3050 50  0001 L BNN "Field4"
+F 5 "A" H 3450 3050 50  0001 L BNN "Field5"
+	1    3450 3050
+	1    0    0    -1
+$EndComp
+$Comp
+L power:GND #PWR0117
+U 1 1 5F486E4E
+P 2600 3600
+F 0 "#PWR0117" H 2600 3350 50  0001 C CNN
+F 1 "GND" H 2605 3427 50  0000 C CNN
+F 2 "" H 2600 3600 50  0001 C CNN
+F 3 "" H 2600 3600 50  0001 C CNN
+	1    2600 3600
+	1    0    0    -1
+$EndComp
+$Comp
+L power:PWR_FLAG #FLG0102
+U 1 1 5F482E55
+P 2900 3600
+F 0 "#FLG0102" H 2900 3675 50  0001 C CNN
+F 1 "PWR_FLAG" H 2900 3773 50  0000 C CNN
+F 2 "" H 2900 3600 50  0001 C CNN
+F 3 "~" H 2900 3600 50  0001 C CNN
+	1    2900 3600
+	-1   0    0    1
+$EndComp
+$Comp
+L power:GND #PWR0116
+U 1 1 5F48215E
+P 2450 2250
+F 0 "#PWR0116" H 2450 2000 50  0001 C CNN
+F 1 "GND" H 2455 2077 50  0000 C CNN
+F 2 "" H 2450 2250 50  0001 C CNN
+F 3 "" H 2450 2250 50  0001 C CNN
+	1    2450 2250
+	1    0    0    -1
+$EndComp
+$Comp
+L Device:C_Small C1
+U 1 1 5F4810C0
+P 2450 2150
+F 0 "C1" H 2542 2196 50  0000 L CNN
+F 1 "1uF" H 2542 2105 50  0000 L CNN
+F 2 "Capacitor_SMD:C_0805_2012Metric_Pad1.15x1.40mm_HandSolder" H 2450 2150 50  0001 C CNN
+F 3 "~" H 2450 2150 50  0001 C CNN
+	1    2450 2150
+	1    0    0    -1
+$EndComp
+Text GLabel 2800 3100 0    50   Input ~ 0
+D+
+Text GLabel 2800 3300 0    50   Input ~ 0
+D-
+$Comp
+L power:GND #PWR0114
+U 1 1 5F46BE27
+P 2500 2750
+F 0 "#PWR0114" H 2500 2500 50  0001 C CNN
+F 1 "GND" H 2505 2577 50  0000 C CNN
+F 2 "" H 2500 2750 50  0001 C CNN
+F 3 "" H 2500 2750 50  0001 C CNN
+	1    2500 2750
+	1    0    0    -1
+$EndComp
+$Comp
+L Device:R_Small R2
+U 1 1 5F46AD36
+P 2900 2750
+F 0 "R2" V 3100 2750 50  0000 C CNN
+F 1 "5K1" V 3000 2750 50  0000 C CNN
+F 2 "Resistor_SMD:R_0805_2012Metric" H 2900 2750 50  0001 C CNN
+F 3 "~" H 2900 2750 50  0001 C CNN
+	1    2900 2750
+	0    1    1    0
+$EndComp
+$Comp
+L Device:R_Small R1
+U 1 1 5F469DAA
+P 2900 2650
+F 0 "R1" V 2704 2650 50  0000 C CNN
+F 1 "5K1" V 2795 2650 50  0000 C CNN
+F 2 "Resistor_SMD:R_0805_2012Metric" H 2900 2650 50  0001 C CNN
+F 3 "~" H 2900 2650 50  0001 C CNN
+	1    2900 2650
+	0    1    1    0
+$EndComp
 $EndSCHEMATC
